Commit message: feat: redesign 3d world with realistic geospatial terrain, 360 camera, and small passage navigation

File: src/naviguard_description/urdf/sensors.xacro (robot description, xacro)
@@ -185,3 +185,101 @@
     </sensor>
   </gazebo>
+  <!-- ==================== 360 DEGREE PANORAMIC SURROUND CAMERA ==================== -->
+  <xacro:property name="camera_360_mass" value="0.15"/>
+  <link name="camera_360_link">
+    <inertial>
+      <origin xyz="0 0 0" rpy="0 0 0"/>
+      <mass value="${camera_360_mass}"/>
+      <inertia
+        ixx="5e-5" ixy="0.0" ixz="0.0"
+        iyy="5e-5" iyz="0.0"
+        izz="5e-5"/>
+    </inertial>
+    <!-- Mast Riser Pole -->
+    <visual name="mast_riser">
+      <origin xyz="0 0 -0.06" rpy="0 0 0"/>
+      <geometry>
+        <cylinder radius="0.012" length="0.12"/>
+      </geometry>
+      <material name="sensor_mast_black"/>
+    </visual>
+    <!-- 360 Panoramic Sensor Base -->
+    <visual name="camera_360_base">
+      <origin xyz="0 0 0" rpy="0 0 0"/>
+      <geometry>
+        <cylinder radius="0.032" length="0.024"/>
+      </geometry>
+      <material name="camera_blue"/>
+    </visual>
+    <!-- 360 Glass Dome Optics -->
+    <visual name="camera_360_dome">
+      <origin xyz="0 0 0.015" rpy="0 0 0"/>
+      <geometry>
+        <sphere radius="0.028"/>
+      </geometry>
+      <material name="lens_glass"/>
+    </visual>
+    <!-- 4 Surround Optical Lens Facets (Visual) -->
+    <visual name="lens_front">
+      <origin xyz="0.030 0 0.005" rpy="0 ${pi/2} 0"/>
+      <geometry>
+        <cylinder radius="0.008" length="0.008"/>
+      </geometry>
+      <material name="sensor_mast_black"/>
+    </visual>
+    <visual name="lens_back">
+      <origin xyz="-0.030 0 0.005" rpy="0 ${pi/2} 0"/>
+      <geometry>
+        <cylinder radius="0.008" length="0.008"/>
+      </geometry>
+      <material name="sensor_mast_black"/>
+    </visual>
+    <visual name="lens_left">
+      <origin xyz="0 0.030 0.005" rpy="${pi/2} 0 0"/>
+      <geometry>
+        <cylinder radius="0.008" length="0.008"/>
+      </geometry>
+      <material name="sensor_mast_black"/>
+    </visual>
+    <visual name="lens_right">
+      <origin xyz="0 -0.030 0.005" rpy="${pi/2} 0 0"/>
+      <geometry>
+        <cylinder radius="0.008" length="0.008"/>
+      </geometry>
+      <material name="sensor_mast_black"/>
+    </visual>
+  </link>
+  <joint name="camera_360_joint" type="fixed">
+    <parent link="base_link"/>
+    <child link="camera_360_link"/>
+    <origin xyz="0.0 0.0 0.28" rpy="0 0 0"/>
+  </joint>
+  <gazebo reference="camera_360_joint">
+    <preserveFixedJoint>true</preserveFixedJoint>
+  </gazebo>
+  <gazebo reference="camera_360_link">
+    <material>
+      <ambient>0.08 0.22 0.45 1.0</ambient>
+      <diffuse>0.10 0.30 0.60 1.0</diffuse>
+      <specular>0.6 0.6 0.6 1.0</specular>
+    </material>
+    <sensor name="naviguard_360_camera" type="camera">
+      <camera>
+        <horizontal_fov>3.14159265</horizontal_fov>
+        <image>
+          <width>1024</width>
+          <height>256</height>
+          <format>R8G8B8</format>
+        </image>
+        <clip>
+          <near>0.05</near>
+          <far>100.0</far>
+        </clip>
+      </camera>
+      <always_on>1</always_on>
+      <update_rate>20</update_rate>
+      <visualize>false</visualize>
+      <topic>/camera/panorama_image</topic>
+    </sensor>
+  </gazebo>
 </robot>

Commit message: feat: trajectory projection, lidar obstacle detection, standoff goal arrival, and expanded 3D world

File: src/naviguard_description/urdf/sensors.xacro (robot description, xacro)
@@ -284,3 +284,79 @@
     </sensor>
   </gazebo>
+  <!-- ==================== 360 DEGREE LIDAR / RADAR SENSOR ==================== -->
+  <xacro:property name="lidar_mass" value="0.18"/>
+  <link name="lidar_link">
+    <inertial>
+      <origin xyz="0 0 0" rpy="0 0 0"/>
+      <mass value="${lidar_mass}"/>
+      <inertia
+        ixx="1e-4" ixy="0.0" ixz="0.0"
+        iyy="1e-4" iyz="0.0"
+        izz="1e-4"/>
+    </inertial>
+    <collision name="lidar_collision">
+      <origin xyz="0 0 0" rpy="0 0 0"/>
+      <geometry>
+        <cylinder radius="0.040" length="0.050"/>
+      </geometry>
+    </collision>
+    <!-- Lower Mounting Base -->
+    <visual name="lidar_base">
+      <origin xyz="0 0 -0.01" rpy="0 0 0"/>
+      <geometry>
+        <cylinder radius="0.042" length="0.028"/>
+      </geometry>
+      <material name="sensor_mast_black"/>
+    </visual>
+    <!-- Upper Spinning Optical Ring -->
+    <visual name="lidar_dome">
+      <origin xyz="0 0 0.012" rpy="0 0 0"/>
+      <geometry>
+        <cylinder radius="0.038" length="0.022"/>
+      </geometry>
+      <material name="camera_blue"/>
+    </visual>
+  </link>
+  <joint name="lidar_joint" type="fixed">
+    <parent link="base_link"/>
+    <child link="lidar_link"/>
+    <origin xyz="0.10 0.0 0.18" rpy="0 0 0"/>
+  </joint>
+  <gazebo reference="lidar_joint">
+    <preserveFixedJoint>true</preserveFixedJoint>
+  </gazebo>
+  <gazebo reference="lidar_link">
+    <sensor name="naviguard_lidar" type="gpu_lidar">
+      <always_on>1</always_on>
+      <update_rate>15</update_rate>
+      <visualize>true</visualize>
+      <topic>/scan</topic>
+      <ray>
+        <scan>
+          <horizontal>
+            <samples>360</samples>
+            <resolution>1</resolution>
+            <min_angle>-3.14159265</min_angle>
+            <max_angle>3.14159265</max_angle>
+          </horizontal>
+          <vertical>
+            <samples>1</samples>
+            <resolution>1</resolution>
+            <min_angle>0</min_angle>
+            <max_angle>0</max_angle>
+          </vertical>
+        </scan>
+        <range>
+          <min>0.10</min>
+          <max>16.0</max>
+          <resolution>0.01</resolution>
+        </range>
+        <noise>
+          <type>gaussian</type>
+          <mean>0.0</mean>
+          <stddev>0.012</stddev>
+        </noise>
+      </ray>
+    </sensor>
+  </gazebo>
 </robot>
